File: Kyttiludzinator/STM32G070RBTx.kicad_sch (KiCad schematic)
At the start: 32 parts, among them IC201 STM32G070RBT6, J201 Conn_02x07_Odd_Even, SW201 SW_Push, SW202 SW_Push, SW203 SW_Push, SW204 SW_Push, Y201 16MHz

Commit message: Finalversion
Parts:
- J201: footprint Connector_PinHeader_1.27mm:PinHeader_2x07_P1.27mm_Vertical -> Connector_PinHeader_1.27mm:PinHeader_2x07_P1.27mm_Vertical_SMD
- L201: footprint Inductor_SMD:L_0603_1608Metric -> Inductor_SMD:L_0603_1608Metric_Pad1.05x0.95mm_HandSolder
Other:
- note added: "to limited the current"
Changed lines of the file:
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@@
     (effects (font (size 4 4) (thickness 0.8) bold (color 255 0 34 1)) (justify left bottom))
+  )
+  (text "to limited the current \n" (at 139.7 58.42 0)
+    (effects (font (size 1.27 1.27)) (justify left bottom))
   )
   (text "STM32" (at 26.67 27.94 0)
@@
       (effects (font (size 1.27 1.27)) hide)
     )
-    (property "Footprint" "Connector_PinHeader_1.27mm:PinHeader_2x07_P1.27mm_Vertical" (at 237.49 50.8 0)
+    (property "Footprint" "Connector_PinHeader_1.27mm:PinHeader_2x07_P1.27mm_Vertical_SMD" (at 237.49 50.8 0)
       (effects (font (size 1.27 1.27)) hide)
     )
@@
       (effects (font (size 1.27 1.27)))
     )
-    (property "Footprint" "Inductor_SMD:L_0603_1608Metric" (at 92.71 163.83 0)
-      (effects (font (size 1.27 1.27)) hide)
-    )
+    (property "Footprint" "Inductor_SMD:L_0603_1608Metric_Pad1.05x0.95mm_HandSolder" (at 92.71 163.83 0)
+      (effects (font (size 1.27 1.27)) hide)
+    )
