File: Kyttiludzinator/_autosave-Kyttiludzinator.kicad_pcb (KiCad board)
At the start: 4 copper layers, 90 x 70 mm, 82 parts, among them IC201 STM32G070RBT6, IC401 NCS199A2RSQT2G, IC402 NCS199A2RSQT2G, IC501 IIM-20670, J101 Conn_01x06, J102 Conn_01x06, J201 Conn_02x07_Odd_Even, J501 Conn_01x08, J502 Conn_01x03, J505 Conn_01x03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

Commit message: Add files via upload
Parts:
- U101: renamed from Driver motor 1
- moved SW204 39.1 mm to (166.5, 63.3), turned to 180 degrees
- moved SW201 36.2 mm to (166.5, 76.3), turned to 180 degrees
- moved J507 35.3 mm to (184.8, 41.0), turned to 90 degrees
- moved IC501 33.9 mm to (199.0, 82.2), turned to 90 degrees
- moved SW203 31.9 mm to (170.2, 71.0), turned to 180 degrees
- moved SW202 31.8 mm to (170.3, 67.1), turned to 180 degrees
- moved J506 22.7 mm to (212.7, 50.8)
- moved PS301 20.0 mm to (186.6, 78.5)
- moved J201 15.7 mm to (202.2, 53.8), turned to 180 degrees
- moved J505 10.9 mm to (212.7, 60.3)
- moved Y201 7.78 mm to (168.8, 55.8)
Connections:
- C202 pad 2: Net-(C202-Pad2) -> /STM32G070RBT6/OSC_OUT
- IC201 pad 59: Moustache_1 -> Moustache_4
- IC401 pad : +BATT -> (no net)
- IC401 pad 5: +BATT -> Net-(IC401-IN-)
- IC402 pad 4: +BATT -> Net-(IC402-IN+)
- IC402 pad 5: +BATT -> Net-(IC402-IN-)
- J102 pad 1: /Drivers_moteurs/Motor2+ -> /Drivers_moteurs/Motor2-
- J102 pad 6: /Drivers_moteurs/Motor2- -> /Drivers_moteurs/Motor2+
- R101 pad 2: +BATT -> Net-(IC401-IN+)
- R201 pad 2: Net-(C202-Pad2) -> /STM32G070RBT6/OSC_OUT
- R401 pad 2: +BATT -> Net-(IC402-IN+)
- Y201 pad 1: Net-(C202-Pad2) -> /STM32G070RBT6/OSC_OUT
Routing:
- net Moustache_2: track 0.00 -> 27.8 mm
- net /STM32G070RBT6/SWCLK: track 0.00 -> 22.5 mm
- net /STM32G070RBT6/SWDIO: track 0.00 -> 19.5 mm
