File: Kyttiludzinator/_autosave-STM32G070RBTx.kicad_sch (KiCad schematic)
At the start: 32 parts, among them IC201 STM32G070RBT6, J201 Conn_02x07_Odd_Even, SW201 SW_Push, SW202 SW_Push, SW203 SW_Push, SW204 SW_Push, Y201 16MHz

Commit message: Add files via upload
Connections:
- net Moustache_1: no longer IC201.59 (PB5)
- new net Moustache_4: IC201.59 (PB5)
Changed lines of the file:
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@@
     )
   )
-  (global_label "Moustache_1" (shape input) (at 71.12 39.37 90) (fields_autoplaced)
+  (global_label "Moustache_4" (shape input) (at 71.12 39.37 90) (fields_autoplaced)
     (effects (font (size 1.27 1.27) (thickness 0.254) bold) (justify left))
     (property "Intersheetrefs" "${INTERSHEET_REFS}" (at 71.12 23.8803 90)
