File: Kyttiludzinator/Charger.kicad_sch (KiCad schematic)
At the start: 1 part, among them U301 MP1475DJ-LF-P

Commit message: Add files via upload
Parts:
- added Alim_batterie301, Alim_charger301: Conn_01x02, Connector_PinHeader_2.54mm:PinHeader_1x02_P2.54mm_Vertical, symbol Connector_Generic:Conn_01x02
- added C210, C211: 1uF, Capacitor_SMD:C_0603_1608Metric_Pad1.08x0.95mm_HandSolder, symbol Device:C_Small
- added C303, C304, C307: 22uF, Capacitor_SMD:C_0603_1608Metric_Pad1.08x0.95mm_HandSolder, symbol Device:C_Small
- added C305: 15pF, Capacitor_SMD:C_0603_1608Metric_Pad1.08x0.95mm_HandSolder, symbol Device:C_Small
- added C306, C308, C309: 0.1uF, Capacitor_SMD:C_0603_1608Metric_Pad1.08x0.95mm_HandSolder, symbol Device:C_Small
- added D301: 1.5KExxA, Diode_THT:D_DO-201AE_P15.24mm_Horizontal, symbol Diode:1.5KExxA
- added F302: Fuse, symbol Device:Fuse
- added L301: 4.7uF, Capacitor_SMD:C_0603_1608Metric_Pad1.08x0.95mm_HandSolder, symbol Device:L_Small
- added PS201: MIC5317-3.3YM5-TR, Library:SOT95P280X145-5N, symbol Ludzlib:MIC5317-3.3YM5-TR
- added R301: 20, Resistor_SMD:R_0805_2012Metric_Pad1.20x1.40mm_HandSolder, symbol Device:R_Small
- added R302: 16k, Resistor_SMD:R_1206_3216Metric, symbol Device:R_Small
- added R303: 40.2k, Resistor_SMD:R_1206_3216Metric, symbol Device:R_Small
- added R304: 7.36k, Resistor_SMD:R_1206_3216Metric, symbol Device:R_Small
- added R305, R306: 100k, Resistor_SMD:R_0603_1608Metric, symbol Device:R_Small
- added SW301: SW_DP3T, symbol Switch:SW_DP3T
- U301: footprint (none) -> Library:SOT65P280X100-8N
Connections:
- net at U301.1 (PG): now also R306.1
- net +BATT: now reaches U301.2 (IN)
- net +BATT: now also C307.1, C308.1, R305.2, SW301.4
- net at U301.3 (SW): now also C306.1, L301.1
- net at U301.5 (BST): now also R301.1
- net at U301.6 (EN/SYNC): now also R305.1
- net at U301.7 (VCC): now also C309.2, R306.2
- net at U301.8 (FB): now also R302.1
- new net: Alim_batterie301.2 (Pin_2), F302.1
- new net: D301.1 (A1), SW301.1
- new net: F302.2, SW301.3
- new net: Alim_charger301.2 (Pin_2), D301.2 (A2)
- new net: C306.2, R301.2
- new net: C305.1, R302.2, R303.1, R304.2
- new net +3.3V: C211.1, PS201.5 (VOUT)
- new net +5V: C210.1, C303.1, C304.1, C305.2, L301.2, PS201.1 (VIN), R303.2
- new net GND: Alim_batterie301.1 (Pin_1), Alim_charger301.1 (Pin_1), C210.2, C211.2, C303.2, C304.2, C307.2, C308.2, C309.1, PS201.2 (GND), R304.1, SW301.2, U301. (GND)
- no-connect marks 0 -> 1
Other:
- note added: "Alimentation"
- note added: "Regulateur 3.3V"
- title: (none) -> Carte éléctronique Ludzinator

Commit message: Add files via upload
Parts:
- removed F302: Fuse, symbol Device:Fuse
- added F301: Polyfuse, Fuse:Fuse_1206_3216Metric, symbol Device:Polyfuse
- D301: footprint Diode_THT:D_DO-201AE_P15.24mm_Horizontal -> Diode_SMD:D_1206_3216Metric
- L301: value 4.7uF -> 4.7uH; footprint Capacitor_SMD:C_0603_1608Metric_Pad1.08x0.95mm_HandSolder -> Library:INDPM4141X210N
- R302, R303, R304: footprint Resistor_SMD:R_1206_3216Metric -> Resistor_SMD:R_0603_1608Metric_Pad0.98x0.95mm_HandSolder
- R305, R306: footprint Resistor_SMD:R_0603_1608Metric -> Resistor_SMD:R_0603_1608Metric_Pad0.98x0.95mm_HandSolder
- SW301: footprint (none) -> Library:Switch-3
Connections:
- net GND: now also U301.4 (GND); no longer SW301.2, U301. (GND)
- net at Alim_batterie301.2 (Pin_2): now also F301.1
- net at SW301.3: now also F301.2
- no-connect marks 1 -> 2
