File: Kyttiludzinator/Charger.kicad_sch (KiCad schematic)
At the start: 23 parts, among them SW302 Switch, U301 MP1475DJ-LF-P

Commit message: Finalversion
Parts:
- added R307: 100k, Resistor_SMD:R_0603_1608Metric_Pad0.98x0.95mm_HandSolder, symbol Device:R_Small
Connections:
- net +5V: now also R307.2
- net at PS?.3 (EN): now also R307.1
- no-connect marks 1 -> 0
Other:
- note added: "EN HIGHT"
- moved on the sheet: C305
Changed lines of the file:
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@@
   (junction (at 81.28 59.69) (diameter 0) (color 0 0 0 0)
   )
-  (junction (at 106.68 63.5) (diameter 0) (color 0 0 0 0)
+  (junction (at 106.68 64.77) (diameter 0) (color 0 0 0 0)
   )
   (junction (at 39.37 54.61) (diameter 0) (color 0 0 0 0)
@@
   (junction (at 91.44 59.69) (diameter 0) (color 0 0 0 0)
   )
+  (junction (at 185.42 55.88) (diameter 0) (color 0 0 0 0)
+  )
   (junction (at 106.68 59.69) (diameter 0) (color 0 0 0 0)
   )
-  (no_connect (at 185.42 60.96))
   (wire (pts (xy 218.44 63.5) (xy 218.44 64.77))
     (stroke (width 0) (type default))
   )
-  (wire (pts (xy 90.17 63.5) (xy 106.68 63.5))
-    (stroke (width 0) (type default))
-  )
-  (wire (pts (xy 76.2 71.12) (xy 80.01 71.12))
+  (wire (pts (xy 90.17 64.77) (xy 106.68 64.77))
     (stroke (width 0) (type default))
   )
@@
     (stroke (width 0) (type default))
   )
-  (wire (pts (xy 68.58 66.04) (xy 76.2 66.04))
+  (wire (pts (xy 68.58 71.12) (xy 80.01 71.12))
     (stroke (width 0) (type default))
   )
@@
     (stroke (width 0) (type default))
   )
-  (wire (pts (xy 106.68 71.12) (xy 106.68 63.5))
-    (stroke (width 0) (type default))
-  )
-  (wire (pts (xy 179.07 54.61) (xy 179.07 55.88))
+  (wire (pts (xy 106.68 71.12) (xy 106.68 64.77))
     (stroke (width 0) (type default))
   )
@@
     (stroke (width 0) (type default))
   )
-  (wire (pts (xy 106.68 63.5) (xy 106.68 59.69))
-    (stroke (width 0) (type default))
-  )
   (polyline (pts (xy 149.86 11.43) (xy 149.86 102.87))
     (stroke (width 0) (type default))
@@
     (stroke (width 0) (type default))
   )
+  (wire (pts (xy 106.68 59.69) (xy 106.68 64.77))
+    (stroke (width 0) (type default))
+  )
   (wire (pts (xy 184.15 64.77) (xy 179.07 64.77))
     (stroke (width 0) (type default))
@@
     (stroke (width 0) (type default))
   )
-  (wire (pts (xy 76.2 66.04) (xy 76.2 71.12))
+  (wire (pts (xy 179.07 49.53) (xy 179.07 55.88))
     (stroke (width 0) (type default))
   )
@@
     (stroke (width 0) (type default))
   )
-  (wire (pts (xy 90.17 68.58) (xy 90.17 71.12))
+  (wire (pts (xy 68.58 71.12) (xy 68.58 66.04))
+    (stroke (width 0) (type default))
+  )
+  (wire (pts (xy 90.17 69.85) (xy 90.17 71.12))
     (stroke (width 0) (type default))
   )
@@
     (effects (font (size 1.27 1.27)) (justify left bottom))
   )
+  (text "EN HIGHT" (at 189.23 80.01 0)
+    (effects (font (size 1.27 1.27)) (justify left bottom))
+  )
   (text "Step-Down Converter\nInput 7V -> Output 5V" (at 31.75 27.94 0)
     (effects (font (size 4 4) (thickness 0.8) bold (color 255 0 34 1)) (justify left bottom))
@@
     (effects (font (size 1.27 1.27)) (justify left bottom))
   )
-  (text "Bypass C" (at 219.71 69.85 0)
+  (text "Bypass C" (at 213.36 68.58 0)
     (effects (font (size 1.27 1.27)) (justify left bottom))
   )
@@
     )
   )
-  (symbol (lib_id "power:+5V") (at 179.07 54.61 0) (unit 1)
-    (in_bom yes) (on_board yes) (dnp no) (fields_autoplaced)
-    (property "Reference" "#PWR?" (at 179.07 58.42 0)
-      (effects (font (size 1.27 1.27)) hide)
-    )
-    (property "Value" "+5V" (at 179.07 50.8 0)
-      (effects (font (size 1.27 1.27)))
-    )
-    (property "Footprint" "" (at 179.07 54.61 0)
-      (effects (font (size 1.27 1.27)) hide)
-    )
-    (property "Datasheet" "" (at 179.07 54.61 0)
+  (symbol (lib_id "power:+5V") (at 179.07 49.53 0) (unit 1)
+    (in_bom yes) (on_board yes) (dnp no) (fields_autoplaced)
+    (property "Reference" "#PWR?" (at 179.07 53.34 0)
+      (effects (font (size 1.27 1.27)) hide)
+    )
+    (property "Value" "+5V" (at 179.07 45.72 0)
+      (effects (font (size 1.27 1.27)))
+    )
+    (property "Footprint" "" (at 179.07 49.53 0)
+      (effects (font (size 1.27 1.27)) hide)
+    )
+    (property "Datasheet" "" (at 179.07 49.53 0)
       (effects (font (size 1.27 1.27)) hide)
     )
@@
     )
   )
-  (symbol (lib_id "Device:C_Small") (at 90.17 66.04 180) (unit 1)
-    (in_bom yes) (on_board yes) (dnp no) (fields_autoplaced)
-    (property "Reference" "C305" (at 92.71 65.3986 0)
-      (effects (font (size 1.27 1.27)) (justify right))
-    )
-    (property "Value" "15pF" (at 92.71 67.9386 0)
-      (effects (font (size 1.27 1.27)) (justify right))
-    )
-    (property "Footprint" "Capacitor_SMD:C_0603_1608Metric_Pad1.08x0.95mm_HandSolder" (at 90.17 66.04 0)
-      (effects (font (size 1.27 1.27)) hide)
-    )
-    (property "Datasheet" "~" (at 90.17 66.04 0)
+  (symbol (lib_id "Device:C_Small") (at 90.17 67.31 180) (unit 1)
+    (in_bom yes) (on_board yes) (dnp no) (fields_autoplaced)
+    (property "Reference" "C305" (at 92.71 66.6686 0)
+      (effects (font (size 1.27 1.27)) (justify right))
+    )
+    (property "Value" "15pF" (at 92.71 69.2086 0)
+      (effects (font (size 1.27 1.27)) (justify right))
+    )
+    (property "Footprint" "Capacitor_SMD:C_0603_1608Metric_Pad1.08x0.95mm_HandSolder" (at 90.17 67.31 0)
+      (effects (font (size 1.27 1.27)) hide)
+    )
+    (property "Datasheet" "~" (at 90.17 67.31 0)
       (effects (font (size 1.27 1.27)) hide)
     )
@@
         )
       )
+    )
+  )
+  (symbol (lib_id "Device:R_Small") (at 185.42 58.42 180) (unit 1)
+    (in_bom yes) (on_board yes) (dnp no)
+    (property "Reference" "R307" (at 180.34 52.07 0)
+      (effects (font (size 1.27 1.27)) (justify right))
+    )
+    (property "Value" "100k" (at 180.34 54.61 0)
+      (effects (font (size 1.27 1.27)) (justify right))
+    )
+    (property "Footprint" "Resistor_SMD:R_0603_1608Metric_Pad0.98x0.95mm_HandSolder" (at 185.42 58.42 0)
+      (effects (font (size 1.27 1.27)) hide)
+    )
+    (property "Datasheet" "~" (at 185.42 58.42 0)
+      (effects (font (size 1.27 1.27)) hide)
+    )
+    (property "Height" "0603" (at 185.42 58.42 0)
+      (effects (font (size 1.27 1.27)) hide)
+    )
+    (pin "1")
+    (pin "2")
+    (instances
+      (project "Kyttiludzinator"
+        (path "/ae6948d5-1dc0-45d1-b607-44e44d4b2b44/a7615b68-eaec-40b2-84b5-a1a21f69b043"
+          (reference "R307") (unit 1)
+        )
+      )
