File: Kyttiludzinator/Kyttiludzinator.kicad_pcb (KiCad board)
At the start: 4 copper layers, 90 x 70 mm, 82 parts, among them IC201 STM32G070RBT6, IC401 NCS199A2RSQT2G, IC402 NCS199A2RSQT2G, IC501 IIM-20670, J101 Conn_01x06, J102 Conn_01x06, J201 Conn_02x07_Odd_Even, J501 Conn_01x08, J502 Conn_01x03, J505 Conn_01x03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

Commit message: Add files via upload
Parts:
- added F301: Polyfuse, Fuse:Fuse_1206_3216Metric, F.Cu at (134.4, 89.9)
- added L201: 6uH, Inductor_SMD:L_0603_1608Metric_Pad1.05x0.95mm_HandSolder, F.Cu at (167.4, 63.9)
- added SW301: SW_DP3T, Library:Switch-3, F.Cu at (139.4, 78.7)
- D206: footprint Library:SOT65P210X110-6N -> Diode_SMD:D_0603_1608Metric_Pad1.05x0.95mm_HandSolder
- D301: footprint Diode_THT:D_DO-201AE_P15.24mm_Horizontal -> Diode_SMD:D_1206_3216Metric
- L301: value 4.7uF -> 4.7uH; footprint Capacitor_SMD:C_0603_1608Metric_Pad1.08x0.95mm_HandSolder -> Library:INDPM4141X210N
- R204, R205, R206, R207, R208, R209: footprint Resistor_SMD:R_0805_2012Metric -> Resistor_SMD:R_0603_1608Metric_Pad0.98x0.95mm_HandSolder
- R302, R303, R304: footprint Resistor_SMD:R_1206_3216Metric -> Resistor_SMD:R_0603_1608Metric_Pad0.98x0.95mm_HandSolder
- R305, R306: footprint Resistor_SMD:R_0603_1608Metric -> Resistor_SMD:R_0603_1608Metric_Pad0.98x0.95mm_HandSolder
- R401: footprint Resistor_SMD:R_0805_2012Metric -> Resistor_SMD:R_1206_3216Metric_Pad1.30x1.75mm_HandSolder
- RShunt: renamed from R101; footprint Resistor_SMD:R_0805_2012Metric -> Resistor_SMD:R_1206_3216Metric_Pad1.30x1.75mm_HandSolder
- U101: renamed from Driver motor 1
- moved C502 163.0 mm to (208.5, 72.3), turned to 90 degrees
- moved C503 161.0 mm to (207.6, 68.1), turned to -90 degrees
- moved C501 156.1 mm to (202.3, 65.2), turned to -90 degrees
- moved C208 136.7 mm to (198.4, 76.7), turned to 90 degrees
- moved C201 136.6 mm to (194.3, 64.4)
- moved C206 135.5 mm to (196.6, 76.7), turned to 90 degrees
- moved R205 131.6 mm to (186.3, 50.3), turned to 90 degrees
- moved R206 130.5 mm to (184.7, 50.3), turned to 90 degrees
- moved R207 127.4 mm to (181.1, 51.8), turned to 90 degrees
- moved R208 126.7 mm to (179.3, 50.3), turned to 90 degrees
- moved C202 126.6 mm to (182.7, 79.9), turned to 90 degrees
- moved R209 125.5 mm to (177.3, 50.3), turned to 90 degrees
- moved R201 119.3 mm to (184.3, 78.0), turned to 90 degrees
- moved C203 119.2 mm to (174.8, 84.3)
- moved D206 118.5 mm to (177.3, 53.8), turned to -90 degrees
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Connections:
- C202 pad 2: Net-(C202-Pad2) -> /STM32G070RBT6/OSC_OUT
- IC201 pad 59: Moustache_1 -> Moustache_4
- IC401 pad : +BATT -> (no net)
- IC401 pad 5: +BATT -> Net-(IC401-IN-)
- IC402 pad 5: +BATT -> Net-(IC402-IN-)
- J102 pad 1: /Drivers_moteurs/Motor2+ -> /Drivers_moteurs/Motor2-
- J102 pad 6: /Drivers_moteurs/Motor2- -> /Drivers_moteurs/Motor2+
- R201 pad 2: Net-(C202-Pad2) -> /STM32G070RBT6/OSC_OUT
- R401 pad 2: +BATT -> Net-(IC402-IN+)
- U101 pad 2: Net-(U101-VM) -> Net-(IC401-IN-)
- U301 pad 4: (no net) -> GND
- U402 pad 2: Net-(U402-VM) -> Net-(IC402-IN-)
- Y201 pad 1: Net-(C202-Pad2) -> /STM32G070RBT6/OSC_OUT
Routing:
- net PWM_MOT1_CH1: track 0.00 -> 47.1 mm, vias 0 -> 2
- net PWM_MOT1_CH2: track 0.00 -> 44.0 mm, vias 0 -> 2
- net PWM_MOT2_CH1: track 1.24 -> 43.7 mm, vias 1 -> 4
- net PWM_MOT2_CH2: track 1.24 -> 38.7 mm, vias 1 -> 2
- net +5V: track 0.00 -> 32.5 mm
- net SPI1_MISO: track 0.00 -> 31.5 mm
- net SPI1_SCK: track 0.00 -> 27.3 mm
- net SPI1_MOSI: track 0.00 -> 26.3 mm
- net Net-(IC201-PA1): track 0.00 -> 24.4 mm
- net /STM32G070RBT6/BUTTON_2: track 0.00 -> 23.7 mm
- net /STM32G070RBT6/BUTTON_1: track 0.00 -> 23.4 mm
- net LIDAR_RX: track 0.00 -> 23.3 mm
- net Net-(IC201-PA0): track 0.00 -> 23.2 mm
- net LIDAR_PWM: track 0.00 -> 23.1 mm
- net /STM32G070RBT6/SWCLK: track 0.00 -> 22.5 mm
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Other:
- board text added: "Driver motors"
- board text added: "Power regulator"
