File: Kyttiludzinator/Kyttiludzinator.kicad_pcb (KiCad board)
At the start: 4 copper layers, 90 x 70 mm, 109 parts, among them IC201 STM32G070RBT6, IC401 NCS199A2RSQT2G, IC402 NCS199A2RSQT2G, IC501 IIM-20670, J201 Conn_02x07_Odd_Even, J401 Conn_01x06, J402 Conn_01x06, J501 Conn_01x03, J502 Conn_01x03, J503 Conn_01x08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

Commit message: Finalversion
Parts:
- removed J505, J507: Conn_01x03, Connector_JST:JST_XH_B3B-XH-A_1x03_P2.50mm_Vertical
- added C408: 100nF, Capacitor_SMD:C_0603_1608Metric_Pad1.08x0.95mm_HandSolder, F.Cu at (175.0, 97.5)
- added C409: 1uF, Capacitor_SMD:C_0603_1608Metric_Pad1.08x0.95mm_HandSolder, F.Cu at (193.3, 98.1)
- added C410: 1uF, Capacitor_SMD:C_0603_1608Metric_Pad1.08x0.95mm_HandSolder, F.Cu at (180.3, 98.1)
- added C411: 1uF, Capacitor_SMD:C_0603_1608Metric_Pad1.08x0.95mm_HandSolder, F.Cu at (169.4, 98.0)
- added C412: 1uF, Capacitor_SMD:C_0603_1608Metric_Pad1.08x0.95mm_HandSolder, F.Cu at (157.0, 98.0)
- added G***: LOGO, Library:beluga, F.Cu at (152.7, 52.0)
- added J509: Conn_01x04, Connector_JST:JST_XH_S4B-XH-A_1x04_P2.50mm_Horizontal, F.Cu at (213.0, 72.2)
- added R307: 100k, Resistor_SMD:R_0603_1608Metric_Pad0.98x0.95mm_HandSolder, F.Cu at (147.4, 83.4)
- added locked: Conn_01x04, Connector_JST:JST_XH_S4B-XH-A_1x04_P2.50mm_Horizontal, F.Cu at (212.9, 57.3)
- Alim_batterie301, Alim_charger301: footprint Connector_JST:JST_XH_B2B-XH-A_1x02_P2.50mm_Vertical -> Connector_JST:JST_XH_S2B-XH-A-1_1x02_P2.50mm_Horizontal
- C406, C407: footprint Capacitor_SMD:C_0603_1608Metric -> Capacitor_SMD:C_0603_1608Metric_Pad1.08x0.95mm_HandSolder
- J201: footprint Connector_PinHeader_2.54mm:PinHeader_2x07_P2.54mm_Vertical -> Connector_PinHeader_1.27mm:PinHeader_2x07_P1.27mm_Vertical_SMD
- J401, J402: footprint Connector_JST:JST_XH_B6B-XH-A_1x06_P2.50mm_Vertical -> Connector_JST:JST_XH_S6B-XH-A_1x06_P2.50mm_Horizontal
- J501, J502: footprint Connector_JST:JST_XH_B3B-XH-A_1x03_P2.50mm_Vertical -> Connector_JST:JST_XH_S3B-XH-A_1x03_P2.50mm_Horizontal
- J503: footprint Connector_JST:JST_XH_B8B-XH-A_1x08_P2.50mm_Vertical -> Connector_JST:JST_XH_S8B-XH-A_1x08_P2.50mm_Horizontal
- J504, J506: value Conn_01x03 -> Conn_01x04; footprint Connector_JST:JST_XH_B3B-XH-A_1x03_P2.50mm_Vertical -> Connector_JST:JST_XH_S4B-XH-A_1x04_P2.50mm_Horizontal
- L201: footprint Inductor_SMD:L_0603_1608Metric -> Inductor_SMD:L_0603_1608Metric_Pad1.05x0.95mm_HandSolder
- U401, U402: footprint Library:SOIC127P600X175-8N -> Package_SO:SOIC-8-1EP_3.9x4.9mm_P1.27mm_EP2.62x3.51mm_ThermalVias
- moved J506 22.5 mm to (194.4, 42.3), turned to 180 degrees
- moved SW201 20.3 mm to (174.5, 77.5), turned to -90 degrees
- moved D404 17.8 mm to (155.6, 63.5)
- moved REF** 17.8 mm to (158.6, 63.0)
- moved REF** 17.8 mm to (152.7, 63.0)
- moved D404 17.8 mm to (152.7, 65.8)
- moved D404 17.8 mm to (158.6, 65.8)
- moved R404 17.8 mm to (151.8, 68.3)
- moved R404 17.8 mm to (159.6, 68.3)
- moved REF** 17.8 mm to (155.6, 60.3)
- moved R404 17.8 mm to (155.6, 67.2)
- moved C207 15.6 mm to (172.0, 76.8), turned to -90 degrees
- moved L301 13.5 mm to (133.6, 85.9), turned to 90 degrees
- moved F301 12.6 mm to (133.2, 62.1), turned to 0 degrees
- moved C307 12.5 mm to (146.4, 88.0), turned to 180 degrees
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Connections:
- net /Drivers_moteurs/In_1- renamed /Drivers_moteurs/M1_VM
- C401 pad 1: +BATT -> +5V
- C402 pad 1: +BATT -> +5V
- IC401 pad : (no net) -> +BATT
- J401 pad 3: Codeur1_PH1 -> Codeur1_PH2
- J401 pad 4: Codeur1_PH2 -> Codeur1_PH1
- J504 pad 2: Moustache_1 -> +3.3V
- J504 pad 3: +3.3V -> Moustache_1
- J506 pad 1: Moustache_3 -> Moustache_4
- J506 pad 2: Moustache_3 -> +3.3V
- J506 pad 3: +3.3V -> Moustache_4
- PS301 pad 3: unconnected-(PS301-EN-Pad3) -> Net-(PS301-EN)
- REF** pad 1: (no net) -> GND (x2)
- REFe pad 1: (no net) -> GND
- U401 pad 3: +BATT -> +5V
- U401 pad 6: +BATT -> +5V
- U402 pad 3: +BATT -> +5V
- U402 pad 6: +BATT -> +5V
Routing:
- net Net-(U301-SW): track 23.2 -> 9.26 mm
- net Net-(SW302-B): track 19.1 -> 6.20 mm
- net /STM32G070RBT6/NRST: track 56.3 -> 43.5 mm
- net GND: track 73.2 -> 85.5 mm, vias 58 -> 57
- net /STM32G070RBT6/RX: track 49.7 -> 39.0 mm, vias 1 -> 2
- net Net-(U301-PG): track 12.4 -> 2.62 mm
- net /Drivers_moteurs/REF: track 51.1 -> 41.7 mm
- net /STM32G070RBT6/TX: track 47.7 -> 38.4 mm, vias 1 -> 2
- net +5V: track 58.7 -> 67.4 mm, vias 6 -> 13
- net /Drivers_moteurs/Motor1+: track 12.6 -> 4.15 mm, vias 0 -> 2
- net Moustache_1: track 33.0 -> 41.4 mm
- net /Drivers_moteurs/Motor2+: track 12.4 -> 4.69 mm, vias 0 -> 2
- net +BATT: track 49.4 -> 41.9 mm, vias 8 -> 5
- net Moustache_4: track 23.7 -> 29.8 mm
- net +3.3V: track 43.7 -> 37.7 mm
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- added copper zone on B.Cu, net /Drivers_moteurs/Motor1+
- added copper zone on B.Cu, net /Drivers_moteurs/Motor1-
- added copper zone on B.Cu, net /Drivers_moteurs/Motor2+
- added copper zone on B.Cu, net /Drivers_moteurs/Motor2-
Other:
- board text added: "GILLES Baptiste CHARBONNEAU Tom SERVAN Antoine"
- board text added: "KittyLudzinator"
- board text added: "PWM"
