File: Kyttiludzinator/MoteurProjet_sch.kicad_sch (KiCad schematic)
At the start: 12 parts, among them IC401 NCS199A2RSQT2G, IC402 NCS199A2RSQT2G, J101 Conn_01x06, J102 Conn_01x06, U101 ZXBM5210-S

Commit message: Add files via upload
Parts:
- removed U101: ZXBM5210-S, Package_SO:SOIC-8_3.9x4.9mm_P1.27mm, symbol Driver_Motor:ZXBM5210-S
- added C404: 100nF, Capacitor_SMD:C_0603_1608Metric_Pad1.08x0.95mm_HandSolder, symbol Device:C_Small
- added R402, R403: 100k, Resistor_SMD:R_0603_1608Metric_Pad0.98x0.95mm_HandSolder, symbol Device:R_Small
- added U402: ZXBM5210-S, Library:SOIC127P600X175-8N, symbol Driver_Motor:ZXBM5210-S
- C102: footprint (none) -> Capacitor_SMD:C_0603_1608Metric_Pad1.08x0.95mm_HandSolder
- IC401, IC402: footprint SOT65P210X110-6N -> Library:SOT65P210X110-6N
- J101, J102: footprint (none) -> Connector_PinHeader_2.54mm:PinHeader_1x06_P2.54mm_Vertical
- R101: footprint (none) -> Resistor_SMD:R_0805_2012Metric
- U101: footprint Package_SO:SOIC-8_3.9x4.9mm_P1.27mm -> Library:SOIC127P600X175-8N
Connections:
- net Codeur1_- is gone; now on net GND: J101.2 (Pin_2)
- net Codeur2_+ is gone; now on net +5V: J102.5 (Pin_5)
- net Codeur2_- is gone; now on net GND: J102.2 (Pin_2)
- net +3.3V: now also R402.1
- net +BATT: now also U402.3 (VDD), U402.6 (VREF)
- net ADC_1: no longer IC402.6 (OUT)
- net GND: now also C404.2, R403.2, U402.8 (GND)
- net REF: now reaches IC401.1 (REF)
- net REF: now also IC402.1 (REF), C404.1, R402.2, R403.1
- net at R101.4: now also U402.2 (VM)
- net Codeur1_+ renamed +5V
- net Motor1_FWD renamed PWM_MOT1_CH1
- net Motor1_O1 renamed Motor1+
- net Motor1_O2 renamed Motor1-
- net Motor1_REV renamed PWM_MOT1_CH2
- net Motor2_O1 renamed Motor2-
- net Motor2-: now also U402.7 (OUT2)
- net Motor2_O2 renamed Motor2+
- net Motor2+: now also U402.1 (OUT1)
- new net ADC_2: IC402.6 (OUT)
- new net PWM_MOT2_CH1: U402.4 (FWD)
- new net PWM_MOT2_CH2: U402.5 (REV)
Other:
- note added: "1.65V"
- note added: "3A -> max current -> 3V(out) 3V/200=0.015V So R=0.015"
- note added: "Current prob ref"
- note added: "Motor driver 2"
- note added: "Shunt resistor"
- note removed: "Motor drive 2"
- title: (none) -> Carte éléctronique Ludzinator
- moved on the sheet: C102, IC401, IC402, J101, J102, R101, U101

Commit message: Add files via upload
Parts:
- removed R101 (x2): 0.015, Resistor_SMD:R_0805_2012Metric, symbol Device:R_Shunt
- added R401, R404: 0.015, symbol Device:R_Small
Connections:
- net +BATT: now also IC401.4 (IN+), IC402.4 (IN+), R401.1, R404.1
- net at IC401.5 (IN-): now also U101.2 (VM), R404.2
- net at U402.2 (VM): now also IC402.5 (IN-), R401.2
