File: Kyttiludzinator/MoteurProjet_sch.kicad_sch (KiCad schematic)
At the start: 30 parts, among them IC401 NCS199A2RSQT2G, IC402 NCS199A2RSQT2G, U402 ZXBM5210-S

Commit message: Finalversion
Parts:
- C406, C407: footprint Capacitor_SMD:C_0603_1608Metric -> Capacitor_SMD:C_0603_1608Metric_Pad1.08x0.95mm_HandSolder
- U402, U?: footprint Library:SOIC127P600X175-8N -> Package_SO:SOIC-8-1EP_3.9x4.9mm_P1.27mm_EP2.62x3.51mm_ThermalVias
Connections:
- net +5V: now also C?.1, C?.1, U402.3 (VDD), U402.6 (VREF), U?.3 (VDD), U?.6 (VREF)
- net +BATT: no longer C?.1, C?.1, U402.3 (VDD), U402.6 (VREF), U?.3 (VDD), U?.6 (VREF)
- net Codeur1_PH1: now also J?.4 (Pin_4); no longer J?.3 (Pin_3)
- net Codeur1_PH2: now also J?.3 (Pin_3); no longer J?.4 (Pin_4)
- net In_1- renamed M1_VM
Other:
- note added: "Gain 100"
- note removed: "Gain 200"
Changed lines of the file:
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@@
     (rev "GILLES Baptiste")
   )
+  (junction (at 54.61 49.53) (diameter 0) (color 0 0 0 0)
+  )
+  (junction (at 97.79 173.99) (diameter 0) (color 0 0 0 0)
+  )
+  (junction (at 73.66 57.15) (diameter 0) (color 0 0 0 0)
+  )
+  (junction (at 97.79 165.1) (diameter 0) (color 0 0 0 0)
+  )
+  (junction (at 77.47 147.32) (diameter 0) (color 0 0 0 0)
+  )
+  (junction (at 91.44 81.28) (diameter 0) (color 0 0 0 0)
+  )
+  (junction (at 59.69 52.07) (diameter 0) (color 0 0 0 0)
+  )
+  (junction (at 203.2 135.89) (diameter 0) (color 0 0 0 0)
+  )
+  (junction (at 54.61 63.5) (diameter 0) (color 0 0 0 0)
+  )
+  (junction (at 58.42 149.86) (diameter 0) (color 0 0 0 0)
+  )
+  (junction (at 91.44 72.39) (diameter 0) (color 0 0 0 0)
+  )
+  (junction (at 116.84 127) (diameter 0) (color 0 0 0 0)
+  )
+  (junction (at 59.69 57.15) (diameter 0) (color 0 0 0 0)
+  )
   (junction (at 58.42 139.7) (diameter 0) (color 0 0 0 0)
   )
-  (junction (at 97.79 173.99) (diameter 0) (color 0 0 0 0)
-  )
-  (junction (at 73.66 57.15) (diameter 0) (color 0 0 0 0)
-  )
-  (junction (at 59.69 49.53) (diameter 0) (color 0 0 0 0)
-  )
-  (junction (at 97.79 165.1) (diameter 0) (color 0 0 0 0)
-  )
-  (junction (at 77.47 147.32) (diameter 0) (color 0 0 0 0)
-  )
-  (junction (at 91.44 81.28) (diameter 0) (color 0 0 0 0)
-  )
-  (junction (at 59.69 52.07) (diameter 0) (color 0 0 0 0)
-  )
-  (junction (at 203.2 135.89) (diameter 0) (color 0 0 0 0)
-  )
-  (junction (at 54.61 63.5) (diameter 0) (color 0 0 0 0)
-  )
-  (junction (at 58.42 149.86) (diameter 0) (color 0 0 0 0)
-  )
-  (junction (at 91.44 72.39) (diameter 0) (color 0 0 0 0)
-  )
-  (junction (at 116.84 127) (diameter 0) (color 0 0 0 0)
-  )
-  (junction (at 62.23 139.7) (diameter 0) (color 0 0 0 0)
-  )
-  (junction (at 59.69 57.15) (diameter 0) (color 0 0 0 0)
-  )
-  (junction (at 54.61 49.53) (diameter 0) (color 0 0 0 0)
-  )
   (junction (at 119.38 147.32) (diameter 0) (color 0 0 0 0)
   )
@@
     (stroke (width 0) (type default))
   )
-  (wire (pts (xy 58.42 139.7) (xy 62.23 139.7))
-    (stroke (width 0) (type default))
-  )
   (wire (pts (xy 88.9 147.32) (xy 88.9 151.13))
     (stroke (width 0) (type default))
@@
     (stroke (width 0) (type default))
   )
-  (wire (pts (xy 59.69 49.53) (xy 59.69 52.07))
-    (stroke (width 0) (type default))
-  )
   (wire (pts (xy 170.18 49.53) (xy 156.21 49.53))
     (stroke (width 0) (type default))
@@
     (stroke (width 0) (type default))
   )
-  (wire (pts (xy 59.69 34.29) (xy 59.69 49.53))
+  (wire (pts (xy 59.69 34.29) (xy 59.69 52.07))
     (stroke (width 0) (type default))
   )
@@
   )
   (wire (pts (xy 77.47 148.59) (xy 77.47 147.32))
-    (stroke (width 0) (type default))
-  )
-  (wire (pts (xy 54.61 49.53) (xy 59.69 49.53))
     (stroke (width 0) (type default))
   )
@@
     (effects (font (size 0.7 0.7)) (justify left bottom))
   )
-  (text "Gain 200" (at 105.41 153.67 0)
+  (text "Gain 100\n" (at 105.41 153.67 0)
     (effects (font (size 1.27 1.27) bold) (justify left bottom))
   )
-  (text "Gain 200" (at 104.14 63.5 0)
+  (text "Gain 100" (at 104.14 63.5 0)
     (effects (font (size 1.27 1.27) bold) (justify left bottom))
   )
@@
   )
   (label "M1_VM" (at 59.69 63.5 90) (fields_autoplaced)
-    (effects (font (size 1.27 1.27)) (justify left bottom))
-  )
-  (label "In_1-" (at 72.39 57.15 0) (fields_autoplaced)
     (effects (font (size 1.27 1.27)) (justify left bottom))
   )
@@
     )
   )
-  (global_label "Codeur1_PH2" (shape input) (at 170.18 54.61 180) (fields_autoplaced)
-    (effects (font (size 1.27 1.27)) (justify right))
-    (property "Intersheetrefs" "${INTERSHEET_REFS}" (at 154.6159 54.61 0)
-      (effects (font (size 1.27 1.27)) (justify right) hide)
-    )
-  )
   (global_label "PWM_MOT1_CH1" (shape input) (at 27.94 33.02 90) (fields_autoplaced)
     (effects (font (size 1.27 1.27) bold) (justify left))
@@
     )
   )
+  (global_label "Codeur1_PH1" (shape input) (at 170.18 54.61 180) (fields_autoplaced)
+    (effects (font (size 1.27 1.27)) (justify right))
+    (property "Intersheetrefs" "${INTERSHEET_REFS}" (at 154.6159 54.61 0)
+      (effects (font (size 1.27 1.27)) (justify right) hide)
+    )
+  )
   (global_label "Codeur2_PH2" (shape input) (at 248.92 57.15 180) (fields_autoplaced)
     (effects (font (size 1.27 1.27)) (justify right))
@@
     )
   )
-  (global_label "Codeur1_PH1" (shape input) (at 170.18 52.07 180) (fields_autoplaced)
+  (global_label "Codeur1_PH2" (shape input) (at 170.18 52.07 180) (fields_autoplaced)
     (effects (font (size 1.27 1.27)) (justify right))
     (property "Intersheetrefs" "${INTERSHEET_REFS}" (at 154.6159 52.07 0)
@@
     )
   )
+  (symbol (lib_id "power:+5V") (at 58.42 139.7 0) (unit 1)
+    (in_bom yes) (on_board yes) (dnp no) (fields_autoplaced)
+    (property "Reference" "#PWR0432" (at 58.42 143.51 0)
+      (effects (font (size 1.27 1.27)) hide)
+    )
+    (property "Value" "+5V" (at 58.42 135.89 0)
+      (effects (font (size 1.27 1.27)))
+    )
+    (property "Footprint" "" (at 58.42 139.7 0)
+      (effects (font (size 1.27 1.27)) hide)
+    )
+    (property "Datasheet" "" (at 58.42 139.7 0)
+      (effects (font (size 1.27 1.27)) hide)
+    )
+    (pin "1")
+    (instances
+      (project "Kyttiludzinator"
+        (path "/ae6948d5-1dc0-45d1-b607-44e44d4b2b44/29ef3ad0-9a27-4625-86ca-e3237d209475"
+          (reference "#PWR0432") (unit 1)
+        )
+      )
+    )
+  )
   (symbol (lib_id "Device:C_Small") (at 38.1 52.07 0) (unit 1)
     (in_bom yes) (on_board yes) (dnp no)
@@
         (path "/ae6948d5-1dc0-45d1-b607-44e44d4b2b44/29ef3ad0-9a27-4625-86ca-e3237d209475"
           (reference "#PWR0408") (unit 1)
+        )
+      )
+    )
+  )
+  (symbol (lib_id "power:+5V") (at 54.61 49.53 0) (unit 1)
+    (in_bom yes) (on_board yes) (dnp no) (fields_autoplaced)
+    (property "Reference" "#PWR0431" (at 54.61 53.34 0)
+      (effects (font (size 1.27 1.27)) hide)
+    )
+    (property "Value" "+5V" (at 54.61 45.72 0)
+      (effects (font (size 1.27 1.27)))
+    )
+    (property "Footprint" "" (at 54.61 49.53 0)
+      (effects (font (size 1.27 1.27)) hide)
+    )
+    (property "Datasheet" "" (at 54.61 49.53 0)
+      (effects (font (size 1.27 1.27)) hide)
+    )
+    (pin "1")
+    (instances
+      (project "Kyttiludzinator"
+        (path "/ae6948d5-1dc0-45d1-b607-44e44d4b2b44/29ef3ad0-9a27-4625-86ca-e3237d209475"
+          (reference "#PWR0431") (unit 1)
         )
       )
@@
       (effects (font (size 1.27 1.27)) (justify left))
     )
-    (property "Footprint" "Library:SOIC127P600X175-8N" (at 62.23 171.45 0)
+    (property "Footprint" "Package_SO:SOIC-8-1EP_3.9x4.9mm_P1.27mm_EP2.62x3.51mm_ThermalVias" (at 62.23 171.45 0)
       (effects (font (size 1.27 1.27)) hide)
     )
@@
       (effects (font (size 1.27 1.27)) (justify left))
     )
-    (property "Footprint" "Library:SOIC127P600X175-8N" (at 58.42 81.28 0)
+    (property "Footprint" "Package_SO:SOIC-8-1EP_3.9x4.9mm_P1.27mm_EP2.62x3.51mm_ThermalVias" (at 58.42 81.28 0)
       (effects (font (size 1.27 1.27)) hide)
     )
@@
       (effects (font (size 1.27 1.27)) (justify left))
     )
-    (property "Footprint" "Capacitor_SMD:C_0603_1608Metric" (at 77.47 151.13 0)
+    (property "Footprint" "Capacitor_SMD:C_0603_1608Metric_Pad1.08x0.95mm_HandSolder" (at 77.47 151.13 0)
       (effects (font (size 1.27 1.27)) hide)
     )
@@
       (effects (font (size 1.27 1.27)) (justify left))
     )
-    (property "Footprint" "Capacitor_SMD:C_0603_1608Metric" (at 73.66 60.96 0)
-      (effects (font (size 1.27 1.27)) hide)
-    )
+    (property "Footprint" "Capacitor_SMD:C_0603_1608Metric_Pad1.08x0.95mm_HandSolder" (at 73.66 60.96 0)
+      (effects (font (size 1.27 1.27)) hide)
+    )
