File: Kyttiludzinator/Kyttiludzinator.kicad_sch (KiCad schematic)
At the start: 0 parts

Commit message: version Antoine 21-09-23
Other:
- added sheet Moustache (Moustache.kicad_sch)
Changed lines of the file:
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@@
+    )
+  )
+  (sheet (at 62.23 123.19) (size 53.34 30.48) (fields_autoplaced)
+    (stroke (width 0.1524) (type solid))
+    (fill (color 0 0 0 0.0000))
+    (property "Sheetname" "Moustache" (at 62.23 122.4784 0)
+      (effects (font (size 1.27 1.27)) (justify left bottom))
+    )
+    (property "Sheetfile" "Moustache.kicad_sch" (at 62.23 154.2546 0)
+      (effects (font (size 1.27 1.27)) (justify left top))
+    )
+    (instances
+      (project "Kyttiludzinator"
+        (path "/ae6948d5-1dc0-45d1-b607-44e44d4b2b44" (page "5"))
+      )
     )
   )

Commit message: Add files via upload
Other:
- sheet Charger renamed Alimentation
- sheet Driver_moteur renamed Drivers_moteurs
- sheet Moustache renamed Capteurs et IMU
- sheet STM32G070RBTx renamed STM32G070RBT6
- note added: "Ludzinator"
Changed lines of the file:
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@@
     (rev "GILLES Baptiste")
   )
-  (sheet (at 149.86 36.83) (size 48.26 49.53) (fields_autoplaced)
+  (text "Ludzinator" (at 133.35 21.59 0)
+    (effects (font (size 4 4) (thickness 0.8) bold) (justify left bottom))
+  )
+  (sheet (at 173.99 87.63) (size 83.82 73.66) (fields_autoplaced)
     (stroke (width 0.1524) (type solid))
-    (fill (color 0 0 0 0.0000))
-    (property "Sheetname" "Driver_moteur" (at 149.86 36.1184 0)
-      (effects (font (size 1.27 1.27)) (justify left bottom))
+    (fill (color 255 7 219 1.0000))
+    (property "Sheetname" "Drivers_moteurs" (at 173.99 85.5534 0)
+      (effects (font (size 4 4) bold) (justify left bottom))
     )
-    (property "Sheetfile" "MoteurProjet_sch.kicad_sch" (at 149.86 86.9446 0)
+    (property "Sheetfile" "MoteurProjet_sch.kicad_sch" (at 173.99 161.8746 0)
       (effects (font (size 1.27 1.27)) (justify left top) hide)
     )
@@
     )
   )
-  (sheet (at 26.67 33.02) (size 46.99 52.07) (fields_autoplaced)
+  (sheet (at 91.44 67.31) (size 71.12 95.25) (fields_autoplaced)
     (stroke (width 0.1524) (type solid))
-    (fill (color 0 0 0 0.0000))
-    (property "Sheetname" "STM32G070RBTx" (at 26.67 32.3084 0)
-      (effects (font (size 1.27 1.27)) (justify left bottom))
+    (fill (color 78 4 255 1.0000))
+    (property "Sheetname" "STM32G070RBT6" (at 91.44 65.2334 0)
+      (effects (font (size 4 4) bold) (justify left bottom))
     )
-    (property "Sheetfile" "STM32G070RBTx.kicad_sch" (at 26.67 85.6746 0)
+    (property "Sheetfile" "STM32G070RBTx.kicad_sch" (at 91.44 163.1446 0)
       (effects (font (size 1.27 1.27)) (justify left top))
     )
@@
     )
   )
-  (sheet (at 85.09 36.83) (size 41.91 48.26) (fields_autoplaced)
+  (sheet (at 24.13 41.91) (size 54.61 60.96) (fields_autoplaced)
     (stroke (width 0.1524) (type solid))
-    (fill (color 0 0 0 0.0000))
-    (property "Sheetname" "Charger" (at 85.09 36.1184 0)
-      (effects (font (size 1.27 1.27)) (justify left bottom))
+    (fill (color 255 1 22 1.0000))
+    (property "Sheetname" "Alimentation" (at 24.13 39.8334 0)
+      (effects (font (size 4 4) bold) (justify left bottom))
     )
-    (property "Sheetfile" "Charger.kicad_sch" (at 85.09 85.6746 0)
+    (property "Sheetfile" "Charger.kicad_sch" (at 24.13 103.4546 0)
       (effects (font (size 1.27 1.27)) (justify left top))
     )
@@
     )
   )
-  (sheet (at 62.23 123.19) (size 53.34 30.48) (fields_autoplaced)
+  (sheet (at 22.86 120.65) (size 66.04 41.91) (fields_autoplaced)
     (stroke (width 0.1524) (type solid))
-    (fill (color 0 0 0 0.0000))
-    (property "Sheetname" "Moustache" (at 62.23 122.4784 0)
-      (effects (font (size 1.27 1.27)) (justify left bottom))
+    (fill (color 39 255 0 1.0000))
+    (property "Sheetname" "Capteurs et IMU" (at 22.86 118.5734 0)
+      (effects (font (size 4 4) bold) (justify left bottom))
     )
-    (property "Sheetfile" "Moustache.kicad_sch" (at 62.23 154.2546 0)
+    (property "Sheetfile" "Moustache.kicad_sch" (at 22.86 163.1446 0)
       (effects (font (size 1.27 1.27)) (justify left top))
     )
