File: Kyttiludzinator/Moustache.kicad_sch (KiCad schematic)
At the start: 11 parts, among them IC501 IIM-20670, J501 Conn_01x03, J502 Conn_01x03, J508 Conn_01x04, J509 Conn_01x04, J510 Conn_01x04, J511 Conn_01x04

Commit message: Finalversion
Parts:
- removed J508, J510, J511: Conn_01x04, symbol Connector_Generic:Conn_01x04
- added J504, J505, J506: Conn_01x04, Connector_JST:JST_XH_S4B-XH-A_1x04_P2.50mm_Horizontal, symbol Connector_Generic:Conn_01x04
- J509: footprint (none) -> Connector_JST:JST_XH_S4B-XH-A_1x04_P2.50mm_Horizontal
Connections:
- net +3.3V: now also J509.2 (Pin_2), J504.2 (Pin_2), J504.4 (Pin_4), J505.2 (Pin_2), J505.4 (Pin_4), J506.2 (Pin_2), J506.4 (Pin_4); no longer J509.3 (Pin_3)
- net Moustache_1: now also J504.1 (Pin_1), J504.3 (Pin_3)
- net Moustache_2: now also J509.3 (Pin_3); no longer J509.2 (Pin_2)
- net Moustache_3: now also J505.1 (Pin_1), J505.3 (Pin_3)
- net Moustache_4: now also J506.1 (Pin_1), J506.3 (Pin_3)
