File: Ludz-le-chat-main/Kyttiludzinator/Kyttiludzinator.kicad_pcb (KiCad board)
At the start: 4 copper layers, 90 x 70 mm, 109 parts, among them IC201 STM32G070RBT6, IC401 NCS199A2RSQT2G, IC402 NCS199A2RSQT2G, IC501 IIM-20670, J201 Conn_02x07_Odd_Even, J401 Conn_01x06, J402 Conn_01x06, J501 Conn_01x03, J502 Conn_01x03, J503 Conn_01x08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

Commit message: Ajout du logo beluga
Parts:
- removed the G*** at (152.5, 66.8)
- added G***: LOGO, logos:chat, F.Cu at (155.2, 53.8)

Commit message: MAJ LOGO
Parts:
- added G***: LOGO, logos:ENSEA, B.Cu at (172.9, 71.2)
Other:
- board text added: "05/10/2023"
- board text added: "GILLES SERVAN CHARBONNEAU"

Commit message: modif connecteur
Parts:
- J201: footprint Connector_PinHeader_2.54mm:PinHeader_2x07_P2.54mm_Vertical -> Connector_PinHeader_1.27mm:PinHeader_2x07_P1.27mm_Vertical_SMD
- moved J201 11.4 mm to (201.3, 44.7)
Routing:
- net /STM32G070RBT6/SWDIO: track 17.6 -> 24.1 mm
- net /STM32G070RBT6/SWCLK: track 19.5 -> 24.8 mm
- net GND: track 73.2 -> 77.8 mm, vias 58 -> 61
- net /STM32G070RBT6/NRST: track 56.3 -> 58.4 mm, vias 2 -> 3
- net /STM32G070RBT6/RX: track 49.7 -> 51.0 mm, vias 1 -> 2
- net /STM32G070RBT6/TX: track 47.7 -> 48.9 mm, vias 1 -> 2
