File: Ludz-le-chat-main/Kyttiludzinator/STM32G070RBTx.kicad_sch (KiCad schematic)
At the start: 32 parts, among them IC201 STM32G070RBT6, J201 Conn_02x07_Odd_Even, SW201 SW_Push, SW202 SW_Push, SW203 SW_Push, SW204 SW_Push, Y201 16MHz

Commit message: modif connecteur
Parts:
- J201: footprint Connector_PinHeader_2.54mm:PinHeader_2x07_P2.54mm_Vertical -> Connector_PinHeader_1.27mm:PinHeader_2x07_P1.27mm_Vertical_SMD
Changed lines of the file:
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@@
       (effects (font (size 1.27 1.27)) hide)
     )
-    (property "Footprint" "Connector_PinHeader_2.54mm:PinHeader_2x07_P2.54mm_Vertical" (at 237.49 50.8 0)
+    (property "Footprint" "Connector_PinHeader_1.27mm:PinHeader_2x07_P1.27mm_Vertical_SMD" (at 237.49 50.8 0)
       (effects (font (size 1.27 1.27)) hide)
     )
